Commit message: update: add bbox support

File: test_data/102145/mobility.urdf (robot description, URDF)
Before this commit: robot partnet_007cedc3-0ea3-4138-8311-7dd457c86b51, 6 links, 5 joints
Joints:
- joint joint_0: limit lower=-0.6094689747964199 upper=0.28274333882308117 -> lower=-0.6094689747964199 upper=0.28274333882308117 effort=30
- joint joint_1: limit lower=0 upper=0.03600000000000003 -> lower=0 upper=0.03600000000000003 effort=30
- joint joint_2: limit lower=0 upper=0.01 -> lower=0 upper=0.01 effort=30

File: test_data/47645/mobility.urdf (robot description, URDF)
Before this commit: robot partnet_985eb4a8f9914873738e43095496b061, 3 links, 2 joints
Joints:
- joint joint_0: limit lower=0.0 upper=3.141592653589793 -> lower=0.0 upper=3.141592653589793 effort=30 velocity=1.0
